File: Garagensteuerung2/Garagensteuerung2.kicad_pcb (KiCad board)
At the start: 2 copper layers, 214.4 x 102.3 mm, 67 parts, among them J1 Conn_LidEnd, J10 Conn_Temp, J11 OLED Oben, J12 OLED Unten, J13 Jumper, J14 Conn_Gate, J15 Conn_LedLid, J16 Conn_DoorFront, J17 Conn_BtnLight, J18 Conn_BtnGate, J19 Conn_BtnLid, J2 Conn_DoorBack, J20 Conn_BtnUp, J21 Conn_BtnRight, J22 Conn_BtnDown, J23 Conn_BtnLeft, J24 Conn_BtnOkay, J3 Conn_Motion, J4 Conn_Radio, J5 Conn_Voltage, J6 Conn_D-Sub-Backend, J7 Conn_Relais, J8 Conn_D-Sub-Handheld, Q1 MMBT3904, Q2 MMBT3904, Q3 MMBT3904, Q4 MMBT3904, Q5 MMBT3904, U3 P82B715DR, U4 MCP23017_SO, U5 P82B715DR, U6 MCP23017_SO

Commit message: Verbesserungen in der Platine einarbeiten
Parts:
- added Q6: MMBT3904, Package_TO_SOT_SMD:SOT-23, F.Cu at (238.9, 51.4)
- added R22: 2k2, Resistor_SMD:R_1206_3216Metric_Pad1.30x1.75mm_HandSolder, F.Cu at (233.4, 50.0)
- added R3: 4k7, Resistor_SMD:R_1206_3216Metric_Pad1.30x1.75mm_HandSolder, F.Cu at (156.8, 47.9)
- added R4: 4k7, Resistor_SMD:R_1206_3216Metric_Pad1.30x1.75mm_HandSolder, F.Cu at (156.8, 51.1)
- added R5: 470, Resistor_SMD:R_1206_3216Metric_Pad1.30x1.75mm_HandSolder, F.Cu at (156.8, 54.4)
- added R6: 470, Resistor_SMD:R_1206_3216Metric_Pad1.30x1.75mm_HandSolder, F.Cu at (156.8, 57.7)
- added R7: 470, Resistor_SMD:R_1206_3216Metric_Pad1.30x1.75mm_HandSolder, F.Cu at (156.8, 61.0)
- added R8: 470, Resistor_SMD:R_1206_3216Metric_Pad1.30x1.75mm_HandSolder, F.Cu at (156.8, 64.3)
Connections:
- J13 pad 2: Net-(J13-Pin_2) -> unconnected-(J13-Pin_2-Pad2)
- J15 pad 2: LedLid -> Net-(J15-Pin_2)
- U6 pad 8: Net-(J13-Pin_2) -> Net-(U6-GPB7)
Routing:
- net LedLid: track 22.1 -> 7.74 mm
- net Net-(J13-Pin_2): track 7.18 -> 0.00 mm
- net (no net): track 0.00 -> 7.18 mm
- net Net-(J15-Pin_2): track 0.00 -> 3.90 mm
- net Net-(Q6-B): track 0.00 -> 3.11 mm
