File: Garagensteuerung2/Garagensteuerung2.kicad_sch (KiCad schematic)
At the start: 73 parts, among them J1 Conn_LidEnd, J10 Conn_Temp, J11 OLED Oben, J12 OLED Unten, J13 Jumper, J14 Conn_Gate, J15 Conn_LedLid, J16 Conn_DoorFront, J17 Conn_BtnLight, J18 Conn_BtnGate, J19 Conn_BtnLid, J2 Conn_DoorBack, J20 Conn_BtnUp, J21 Conn_BtnRight, J22 Conn_BtnDown, J23 Conn_BtnLeft, J24 Conn_BtnOkay, J3 Conn_Motion, J4 Conn_Radio, J5 Conn_Voltage, J6 Conn_D-Sub-Backend, J7 Conn_Relais, J8 Conn_D-Sub-Handheld, Q1 MMBT3904, Q2 MMBT3904, Q3 MMBT3904, Q4 MMBT3904, Q5 MMBT3904, U3 P82B715DR, U4 MCP23017_SO, U5 P82B715DR, U6 MCP23017_SO

Commit message: Verbesserungen in der Platine einarbeiten
Parts:
- added Q6: MMBT3904, Package_TO_SOT_SMD:SOT-23, symbol Transistor_BJT:MMBT3904
- added R22: 470, Resistor_SMD:R_1206_3216Metric_Pad1.30x1.75mm_HandSolder, symbol Device:R
- added R30, R31, R32, R33, R34, R35, R36, R37, R38: 2k2, Resistor_SMD:R_1206_3216Metric_Pad1.30x1.75mm_HandSolder, symbol Device:R
- R23, R24, R25, R26, R27: value 2k2 -> 470
Connections:
- net +3.3VA: now also R30.2, R31.2, R32.2, R33.2, R34.2, R35.2, R36.2, R37.2, R38.2
- net GND1: now also Q6.2 (E)
- net LedLid: no longer J15.2 (Pin_2)
- net at J17.1 (Pin_1), U6.21 (GPA0): now also R31.1
- net at J22.1 (Pin_1), U6.26 (GPA5): now also R36.1
- net at J19.1 (Pin_1), U6.23 (GPA2): now also R33.1
- net at J16.1 (Pin_1), U6.7 (GPB6): now also R30.1
- net at J20.1 (Pin_1), U6.24 (GPA3): now also R34.1
- net at J18.1 (Pin_1), U6.22 (GPA1): now also R32.1
- net at J24.1 (Pin_1), U6.28 (GPA7): now also R38.1
- net at J21.1 (Pin_1), U6.25 (GPA4): now also R35.1
- net at J23.1 (Pin_1), U6.27 (GPA6): now also R37.1
- net at U6.8 (GPB7): now also R22.1; no longer J13.2 (Pin_2)
- new net: Q6.1 (B), R22.2
- new net: J15.2 (Pin_2), Q6.3 (C)
- no-connect marks 13 -> 15
